File: chargeur_de_téléphone.kicad_sch (KiCad schematic)
At the start: 0 parts

Commit message: Adding Gerber folder
Parts:
- added C1: C_Polarized, symbol Device:C_Polarized
- added D2, D3: 1N4148WT, Diode_SMD:D_SOD-523, symbol Diode:1N4148WT
- added D4: LED, symbol Device:LED
- added J1: Screw_Terminal_01x02, symbol Connector:Screw_Terminal_01x02
- added R1, R2, R3, R4: R, symbol Device:R
- added U2: LM317L_SOT-89, Package_TO_SOT_SMD:SOT-89-3, symbol Regulator_Linear:LM317L_SOT-89
Connections:
- new net: R1.1, R2.1, R3.2, U2.1 (ADJ)
- new net: C1.2, D4.1 (K), J1.1 (Pin_1), R1.2, R2.2
- new net: D2.2 (A), R3.1, R4.1, U2.2 (VO)
- new net: D4.2 (A), R4.2
- new net: D3.2 (A), J1.2 (Pin_2)
- new net: C1.1, D2.1 (K), D3.1 (K), U2.3 (VI)
