File: génératrice_musculaire.kicad_sch (KiCad schematic)
At the start: 7 parts, among them J2 CTB0308_2, Q1 XT60_YELLOW, U1 LM2576HVS-12

Commit message: Adding Gerber folder
Parts:
- J2: footprint CTB03082 -> CTB0308_2:CTB03082
Changed lines of the file:
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@@
 			)
 		)
-		(property "Footprint" "CTB03082"
+		(property "Footprint" "CTB0308_2:CTB03082"
 			(at 245.11 166.04 0)
 			(effects
